File: PCB/stand/RKD.kicad_pcb (KiCad board)
At the start: 2 copper layers, 100 x 51.5 mm, 112 parts, among them J1 USB_B_Micro, J10 Conn_01x04_Male, J11 Conn_02x06_Odd_Even, J12 Conn_01x06, J13 Conn_01x03, J14 Conn_01x04, J15 Conn_01x04, J2 Conn_02x02_Odd_Even, J3 Conn_02x04_Odd_Even, J4 Conn_02x02_Odd_Even, J5 Conn_02x04_Odd_Even, K1 Key, K2 Key, K3 Key, K4 Key, SW2 SW_DIP_x04, SW3 SW_Push, SW5 SW_Push, U1 W25Q32JV, U2 RP2040, U3 CH9329, U4 AP1117-33, Y1 Crystal 12MHZ HC49, Y2 Crystal_GND24 12MHZ 3225

Commit message: fix pcb
Other:
- board size 100 x 51.5 mm -> 100 x 50 mm
Changed lines of the file:
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@@
     )
   )
-  (gr_line (start 158.5 87) (end 150 87) (layer "B.SilkS") (width 0.15))
-  (gr_line (start 183.5 87) (end 158.5 87) (layer "B.SilkS") (width 0.15))
-  (gr_line (start 90.5 87) (end 150 87) (layer "B.SilkS") (width 0.15))
   (gr_line (start 170.434 50.3428) (end 173.0756 46.5836) (layer "F.SilkS") (width 0.15))
-  (gr_line (start 90.5 87) (end 150 87) (layer "F.SilkS") (width 0.15))
   (gr_line (start 100.6856 43.942) (end 103.3272 47.7266) (layer "F.SilkS") (width 0.15))
-  (gr_line (start 183.5 87) (end 158.5 87) (layer "F.SilkS") (width 0.15))
-  (gr_line (start 158.5 87) (end 150 87) (layer "F.SilkS") (width 0.15))
   (gr_line (start 103.3018 50.1142) (end 100.6602 46.609) (layer "F.SilkS") (width 0.15))
   (gr_line (start 103.3526 45.339) (end 100.6856 41.4782) (layer "F.SilkS") (width 0.15))
   (gr_line (start 173.0502 41.5036) (end 170.434 45.6184) (layer "F.SilkS") (width 0.15))
   (gr_line (start 170.4848 47.9552) (end 173.1772 44.0436) (layer "F.SilkS") (width 0.15))
-  (gr_line (start 90.5 87) (end 90.5 88.474874) (layer "Edge.Cuts") (width 0.1))
   (gr_arc (start 87 40.5) (mid 88.025126 38.025126) (end 90.5 37) (layer "Edge.Cuts") (width 0.1))
   (gr_line (start 183.5 37) (end 90.5 37) (layer "Edge.Cuts") (width 0.1))
   (gr_arc (start 187 83.5) (mid 185.974874 85.974874) (end 183.5 87) (layer "Edge.Cuts") (width 0.1))
+  (gr_line (start 183.5 87) (end 90.5 87) (layer "Edge.Cuts") (width 0.1))
   (gr_line (start 187 83.5) (end 187 40.5) (layer "Edge.Cuts") (width 0.1))
   (gr_arc (start 183.5 37) (mid 185.974874 38.025126) (end 187 40.5) (layer "Edge.Cuts") (width 0.1))
   (gr_line (start 87 40.5) (end 87 83.5) (layer "Edge.Cuts") (width 0.1))
   (gr_arc (start 90.5 87) (mid 88.025126 85.974874) (end 87 83.5) (layer "Edge.Cuts") (width 0.1))
-  (gr_line (start 183.5 87) (end 183.5 88.474874) (layer "Edge.Cuts") (width 0.1))
   (segment (start 140.335 71.8414) (end 140.2336 71.74) (width 0.15) (layer "F.Cu") (net 1))
   (segment (start 145.401414 54.326973) (end 143.340387 56.388) (width 0.15) (layer "F.Cu") (net 1))
