File: PCB/stand/RKD.kicad_sch (KiCad schematic)
At the start: 63 parts, among them J1 USB_B_Micro, J10 Conn_01x04_Male, J11 Conn_02x06_Odd_Even, J12 Conn_01x06, J13 Conn_01x03, J14 Conn_01x04, J15 Conn_01x04, J2 Conn_02x02_Odd_Even, J3 Conn_02x04_Odd_Even, J4 Conn_02x02_Odd_Even, J5 Conn_02x04_Odd_Even, K1 Key, K2 Key, K3 Key, K4 Key, SW2 SW_DIP_x04, SW3 SW_Push, SW5 SW_Push, U1 W25Q32JV, U2 RP2040, U3 CH9329, U4 AP1117-33, Y1 Crystal 12MHZ HC49, Y2 Crystal_GND24 12MHZ 3225

Commit message: fix pcb
Parts:
- U4: value AP1117-33 -> AMS1117-33
Changed lines of the file:
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@@
     (in_bom yes) (on_board yes) (fields_autoplaced)
     (property "Reference" "U4" (id 0) (at 177.8 45.72 0))
-    (property "Value" "AP1117-33" (id 1) (at 177.8 48.26 0))
+    (property "Value" "AMS1117-33" (id 1) (at 177.8 48.26 0))
     (property "Footprint" "Package_TO_SOT_SMD:SOT-223-3_TabPin2" (id 2) (at 177.8 48.26 0)
       (effects (font (size 1.27 1.27)) hide)
@@
     )
     (path "/cb0d88bb-9c4c-4c4d-ad2e-692d2f8e5d90"
-      (reference "U4") (unit 1) (value "AP1117-33") (footprint "Package_TO_SOT_SMD:SOT-223-3_TabPin2")
+      (reference "U4") (unit 1) (value "AMS1117-33") (footprint "Package_TO_SOT_SMD:SOT-223-3_TabPin2")
     )
     (path "/ff4b2401-c0e1-4c1f-9136-1d9dd7534361"
