File: PCB/stand+sdvx/Type-C/RKD.kicad_pcb (KiCad board)
At the start: 2 copper layers, 100 x 94 mm, 144 parts, among them J1 USB_C_Receptacle_USB2.0, J10 Conn_01x04_Male, J11 Conn_02x06_Odd_Even, J12 Conn_01x06, J13 Conn_01x03, J14 Conn_01x04, J15 Conn_01x04, J2 Conn_02x02_Odd_Even, J3 Conn_02x04_Odd_Even, J4 Conn_02x02_Odd_Even, J5 Conn_02x04_Odd_Even, J6 Conn_02x04_Odd_Even, J7 Conn_02x02_Odd_Even, J8 Conn_02x02_Odd_Even, J9 Conn_02x04_Odd_Even, K1 Key, K2 Key, K3 Key, K4 Key, K5 Key, K6 Key, SW2 SW_DIP_x04, SW3 SW_Push, SW5 SW_Push, SW6 RotaryEncoder_Switch, SW7 SW_Push, SW8 RotaryEncoder_Switch, U1 W25Q32JV, U2 RP2040, U3 CH9329, U4 AP1117-33, Y1 Crystal 12MHZ HC49

Commit message: rename
Parts:
- removed kibuzzard-640C98B4: G***, kibuzzard-640C98B4
- added kibuzzard-64E6F17C: G***, kibuzzard-64E6F17C, B.Cu at (157.3, 85.1)
